Commit message: addmove franka

File: panda_table_description/urdf/panda_table.urdf.xacro (robot description, xacro)
@@ -50,5 +50,5 @@
     <visual>
       <geometry>
-	<box size="1.0 1.11 0.7" />
+	<box size="1.0 1.35 0.7" />
       </geometry>
       <origin rpy="0 0 0" xyz="0 0 0.35" />
@@ -56,5 +56,5 @@
     <collision>
       <geometry>
-	<box size="1.0 1.11 0.7" />
+	<box size="1.0 1.35 0.7" />
       </geometry>
       <origin rpy="0 0 0" xyz="0 0 0.35" />
@@ -154,32 +154,32 @@
   </joint>
   <joint name="table_joint" type="fixed">
-    <parent link="table" />
+    <parent link="world" />
     <child link = "mount_flange_link" />
-    <origin xyz="0.0 0.305 0.7" rpy="0.0 0.0 1.5707" />
+    <origin xyz="0.0 0.45 0.7" rpy="0.0 0.0 1.5707" />
   </joint>
   <joint name="table_column1" type="fixed">
     <parent link="table" />
     <child link = "column1" />
-    <origin xyz="0.45 -0.505 0.7" rpy="0.0 0.0 0.0" />
+    <origin xyz="0.45 -0.605 0.7" rpy="0.0 0.0 0.0" />
   </joint>
   <joint name="table_column2" type="fixed">
     <parent link="table" />
     <child link = "column2" />
-    <origin xyz="-0.45 -0.505 0.7" rpy="0.0 0.0 0.0" />
+    <origin xyz="-0.45 -0.605 0.7" rpy="0.0 0.0 0.0" />
   </joint>
   <joint name="table_011_banana" type="fixed">
     <parent link="table" />
     <child link = "011_banana" />
-    <origin xyz="0.0 -0.265 0.45" rpy="0.0 0.0 0.0" />
+    <origin xyz="0.0 0.0 0.45" rpy="0.0 0.0 0.0" />
   </joint>
   <joint name="table_065-h_cups" type="fixed">
     <parent link="table" />
     <child link = "065-h_cups" />
-    <origin xyz="0.10 -0.205 0.45" rpy="0.0 0.0 0.0" />
+    <origin xyz="0.10 0.0 0.45" rpy="0.0 0.0 0.0" />
   </joint>
   <joint name="world_camera_joint" type="fixed">
-    <parent link="world" />
+    <parent link="table" />
     <child link = "camera_link" />
-    <origin xyz="-0.045 -0.85 1.31" rpy="0.0 0.745 1.56" />
+    <origin xyz="0.0 -0.605 1.2" rpy="0.0 ${pi/3.5} ${pi/2}" />
   </joint>
   <link name="asus_rgb_optical_frame"/>

Commit message: add execute grasp

File: panda_table_description/urdf/panda_table.urdf.xacro (robot description, xacro)
@@ -103,5 +103,5 @@
     </collision>
    </link>
-   <link name="011_banana">
+  <link name="011_banana">
     <visual>
       <geometry>
@@ -116,5 +116,47 @@
       <origin rpy="0 0 0" xyz="0.0 0.0 0.2575" />
     </collision>
-   </link>
+  </link>
+  <link name="008_pudding_box">
+    <visual>
+      <geometry>
+	      <mesh filename="package://panda_table_description/meshes/008_pudding_box/textured.dae"/>
+      </geometry>
+      <origin rpy="0 0 0" xyz="0.0 0.0 0.2575" />
+    </visual>
+    <collision>
+      <geometry>
+        <mesh filename="package://panda_table_description/meshes/008_pudding_box/nontextured.stl"/>
+      </geometry>
+      <origin rpy="0 0 0" xyz="0.0 0.0 0.2575" />
+    </collision>
+   </link>
+    <link name="024_bowl">
+    <visual>
+      <geometry>
+	      <mesh filename="package://panda_table_description/meshes/024_bowl/textured.dae"/>
+      </geometry>
+      <origin rpy="0 0 0" xyz="0.0 0.0 0.2575" />
+    </visual>
+    <collision>
+      <geometry>
+        <mesh filename="package://panda_table_description/meshes/024_bowl/nontextured.stl"/>
+      </geometry>
+      <origin rpy="0 0 0" xyz="0.0 0.0 0.2575" />
+    </collision>
+   </link>
+  <link name="044_flat_screwdriver">
+    <visual>
+      <geometry>
+	      <mesh filename="package://panda_table_description/meshes/044_flat_screwdriver/textured.dae"/>
+      </geometry>
+      <origin rpy="0 0 0" xyz="0.0 0.0 0.2575" />
+    </visual>
+    <collision>
+      <geometry>
+        <mesh filename="package://panda_table_description/meshes/044_flat_screwdriver/nontextured.stl"/>
+      </geometry>
+      <origin rpy="0 0 0" xyz="0.0 0.0 0.2575" />
+    </collision>
+  </link>
   <link name="065-h_cups">
     <visual>
@@ -171,10 +213,25 @@
     <parent link="table" />
     <child link = "011_banana" />
+    <origin xyz="0.1 0.0 0.45" rpy="0.0 0.0 0.0" />
+  </joint>
+  <joint name="008_pudding_box" type="fixed">
+    <parent link="table" />
+    <child link = "008_pudding_box" />
+    <origin xyz="0.0 -0.1 0.45" rpy="0.0 0.0 0.0" />
+  </joint>
+  <joint name="024_bowl" type="fixed">
+    <parent link="table" />
+    <child link = "024_bowl" />
+    <origin xyz="-0.13 0.0 0.45" rpy="0.0 0.0 0.0" />
+  </joint>
+  <joint name="044_flat_screwdriver" type="fixed">
+    <parent link="table" />
+    <child link = "044_flat_screwdriver" />
+    <origin xyz="0.0 0.1 0.45" rpy="0.0 0.0 0.0" />
+  </joint>
+  <joint name="table_065-h_cups" type="fixed">
+    <parent link="table" />
+    <child link = "065-h_cups" />
     <origin xyz="0.0 0.0 0.45" rpy="0.0 0.0 0.0" />
-  </joint>
-  <joint name="table_065-h_cups" type="fixed">
-    <parent link="table" />
-    <child link = "065-h_cups" />
-    <origin xyz="0.10 0.0 0.45" rpy="0.0 0.0 0.0" />
   </joint>
   <joint name="world_camera_joint" type="fixed">

Commit message: data generation

File: panda_table_description/urdf/panda_table.urdf.xacro (robot description, xacro)
@@ -186,5 +186,5 @@
     <inertial>
       <mass value="0.316" />
-      <origin xyz="0 0 0" rpy="0 1.56 0"/>
+      <origin xyz="0 0 0" rpy="0 0 0"/>
       <inertia ixx="0.0007765" ixy="0" ixz="0" iyy="0.0000725" iyz="0" izz="0.0007657" />
     </inertial>
@@ -238,5 +238,5 @@
     <parent link="table" />
     <child link = "camera_link" />
-    <origin xyz="0.0 -0.605 1.2" rpy="0.0 ${pi/3.5} ${pi/2}" />
+    <origin xyz="-0.05 -0.40 1.32" rpy="0.0 ${pi/3} ${pi/2}" />
   </joint>
   <link name="asus_rgb_optical_frame"/>

Commit message: cvpr

File: panda_table_description/urdf/panda_table.urdf.xacro (robot description, xacro)
@@ -238,5 +238,5 @@
     <parent link="table" />
     <child link = "camera_link" />
-    <origin xyz="-0.05 -0.40 1.32" rpy="0.0 ${pi/3} ${pi/2}" />
+    <origin xyz="-0.05 -0.60 1.15" rpy="0.0 ${0.255*pi} ${pi/2}" />
   </joint>
   <link name="asus_rgb_optical_frame"/>
